File: _autosave-Energy Harvester Design.kicad_pcb (KiCad board)
At the start: 2 copper layers, 22 parts, among them U1 ADP5091, U2 Nucleo_L432KC

Commit message: Update
Parts:
- moved JP1 186.9 mm to (154.0, 112.5)
- moved RR_PG_HYST1 186.9 mm to (154.0, 109.2)
