File: Energy Harvester Design.kicad_pcb (KiCad board)
At the start: 2 copper layers, 22 parts, among them U1 ADP5091, U2 Nucleo_L432KC

Commit message: Update PCB
Parts:
- added TEG1: ~, Connector_Molex:Molex_Micro-Fit_3.0_43650-0200_1x02_P3.00mm_Horizontal, F.Cu at (120.9, 68.5)
- BT1, BT2: moved to B.Cu
- moved RR_PG_HYST1 139.3 mm to (130.9, 53.1), turned to -90 degrees
- moved JP1 130.5 mm to (122.7, 53.0)
- moved BT2 109.2 mm to (150.9, 47.8), turned to 180 degrees
- moved R_TERM1 72.0 mm to (139.1, 48.0)
- moved R_PG1 59.2 mm to (132.1, 41.2), turned to 180 degrees
- moved R_SD2 54.1 mm to (146.5, 50.5)
- moved BT1 52.5 mm to (151.1, 72.8), turned to 180 degrees
- moved R_BK1 48.4 mm to (138.6, 50.5), turned to 180 degrees
- moved R_BK2 47.9 mm to (135.5, 45.0), turned to 180 degrees
- moved C4 44.8 mm to (146.4, 61.2), turned to -90 degrees
- moved R_TERM2 43.9 mm to (142.9, 48.0)
- moved C1 39.5 mm to (133.1, 65.0), turned to -90 degrees
- moved U2 39.5 mm to (166.8, 57.2), turned to 90 degrees
- moved L1 38.5 mm to (143.9, 65.2), turned to -90 degrees
- moved R1 37.5 mm to (134.6, 49.2), turned to 90 degrees
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Connections:
- net Net-(TEG1-POS_Lead_Wire) renamed /TEG_POS
- C1 pad 2: GNDA -> GND
- R1 pad 1: GNDA -> GND
- R2 pad 1: GNDA -> GND
- R3 pad 1: GNDA -> GND
- R_BK2 pad 2: GNDA -> GND
- R_PG2 pad 2: GNDA -> GND
- R_SD2 pad 2: GNDA -> GND
- R_TERM2 pad 2: GNDA -> GND
- U1 pad 23: GNDA -> GND
Routing:
- net Net-(BT1-+): track 0.00 -> 59.1 mm
- net Net-(U1-LLD): track 0.00 -> 58.0 mm, vias 0 -> 2
- net Net-(U1-REG_D0): track 0.00 -> 50.0 mm, vias 0 -> 2
- net GND: track 0.00 -> 44.6 mm, vias 0 -> 2
- net Net-(U1-PGOOD): track 0.00 -> 37.9 mm, vias 0 -> 1
- net Net-(U1-REG_FB): track 0.00 -> 35.2 mm
- net Net-(U1-TERM): track 0.00 -> 33.6 mm, vias 0 -> 2
- net /TEG_POS: track 0.00 -> 28.9 mm, vias 0 -> 1
- net Net-(U1-REF): track 0.00 -> 24.2 mm, vias 0 -> 2
- net Net-(U1-SETPG): track 0.00 -> 24.0 mm
- net Net-(U1-SETSD): track 0.00 -> 19.0 mm, vias 0 -> 2
- net Net-(U1-SETBK): track 0.00 -> 18.4 mm, vias 0 -> 2
- net Net-(BT2-+): track 0.00 -> 17.6 mm
- net Net-(JP1-B): track 0.00 -> 17.5 mm, vias 0 -> 2
- net Net-(U1-VID): track 0.00 -> 11.4 mm, vias 0 -> 2
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- added copper zone on F.Cu, net GND
Other:
- board outline added: 86 x 66.8 mm
- board text removed: "Talha Haris and Gavin Wang"
