File: Energy Harvester Design.kicad_sch (KiCad schematic)
At the start: 21 parts, among them U1 ADP5091, U2 Nucleo_L432KC

Commit message: Update
Parts:
- added JP1: Jumper_2_Bridged, Jumper:SolderJumper-2_P1.3mm_Bridged_Pad1.0x1.5mm, symbol Jumper:Jumper_2_Bridged
- added R3: 150k, Resistor_SMD:R_0805_2012Metric, symbol Device:R_US
- BT1, BT2: footprint (none) -> Battery:BatteryHolder_Keystone_103_1x20mm
- C1, C2, C3, C4: footprint (none) -> Capacitor_SMD:C_0805_2012Metric
- L1: footprint (none) -> Inductor_SMD:L_0805_2012Metric
- R1, R2, RR_PG_HYST1, R_BK1, R_BK2, R_PG1, R_PG2, R_SD1, R_SD2, R_TERM1, R_TERM2: footprint (none) -> Resistor_SMD:R_0805_2012Metric
- U2: footprint (none) -> UTSVT_Special:NucleoL432KC
Connections:
- net at C3.1, C4.1, U1.14 (REG_OUT)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: no longer U1.24 (REG_D0), U2.23 (A4)
- net at U1.21 (MINOP): now also JP1.2 (B)
- net Earth renamed GND
- net GND: no longer C1.2, R1.1, R2.1, R_BK2.2, R_PG2.2, R_SD2.2, R_TERM2.2, U1.23 (REG_D1)
- new net: RR_PG_HYST1.1, R_PG1.2, U1.5 (SETPG)
- new net: R_BK1.2, R_BK2.1, U1.3 (SETBK)
- new net: R_TERM1.2, R_TERM2.1, U1.4 (TERM)
- new net: JP1.1 (A), R3.2
- new net: U1.24 (REG_D0), U2.23 (A4)
- new net GNDA: C1.2, R1.1, R2.1, R3.1, R_BK2.2, R_PG2.2, R_SD2.2, R_TERM2.2, U1.23 (REG_D1)
- no-connect marks 27 -> 26

Commit message: Update PCB
Parts:
- TEG1: footprint (none) -> Connector_Molex:Molex_Micro-Fit_3.0_43650-0200_1x02_P3.00mm_Horizontal
Connections:
- net GNDA is gone; now on net GND: C1.2, R1.1, R2.1, R3.1, R_BK2.2, R_PG2.2, R_SD2.2, R_TERM2.2, U1.23 (REG_D1)
- net GND: now also TEG1.2 (NEG_TEG); no longer TEG1. (POS_Lead_Wire)
- net TEG_POS: now reaches C2.1, L1.2, U1.10 (VIN)
- net TEG_POS: now also TEG1.1 (POS); no longer TEG1. (POS_Lead_Wire)
Changed lines of the file:
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@@
 	)
 	(junction
-		(at 120.65 60.96)
-		(diameter 0)
-		(color 0 0 0 0)
-	)
-	(junction
 		(at 128.27 60.96)
 		(diameter 0)
@@
 		(color 0 0 0 0)
 	)
+	(junction
+		(at 120.65 60.96)
+		(diameter 0)
+		(color 0 0 0 0)
+	)
 	(no_connect
 		(at 237.49 76.2)
@@
 	(wire
 		(pts
-			(xy 120.65 60.96) (xy 120.65 67.31)
-		)
-		(stroke
-			(width 0)
-			(type default)
-		)
-	)
-	(wire
-		(pts
 			(xy 196.85 129.54) (xy 251.46 129.54)
 		)
@@
 	(wire
 		(pts
+			(xy 120.65 60.96) (xy 120.65 67.31)
+		)
+		(stroke
+			(width 0)
+			(type default)
+		)
+	)
+	(wire
+		(pts
 			(xy 208.28 81.28) (xy 212.09 81.28)
 		)
@@
 	(wire
 		(pts
-			(xy 124.46 49.53) (xy 128.27 49.53)
+			(xy 124.46 46.99) (xy 128.27 46.99)
 		)
 		(stroke
@@
 	(wire
 		(pts
-			(xy 57.15 129.54) (xy 62.23 129.54)
+			(xy 104.14 177.8) (xy 104.14 181.61)
 		)
 		(stroke
@@
 	(wire
 		(pts
-			(xy 107.95 115.57) (xy 104.14 115.57)
+			(xy 57.15 129.54) (xy 62.23 129.54)
 		)
 		(stroke
@@
 	(wire
 		(pts
-			(xy 138.43 85.09) (xy 208.28 85.09)
+			(xy 107.95 115.57) (xy 104.14 115.57)
 		)
 		(stroke
@@
 	(wire
 		(pts
-			(xy 120.65 49.53) (xy 120.65 60.96)
+			(xy 138.43 85.09) (xy 208.28 85.09)
 		)
 		(stroke
@@
 	(wire
 		(pts
+			(xy 90.17 181.61) (xy 90.17 177.8)
+		)
+		(stroke
+			(width 0)
+			(type default)
+		)
+	)
+	(wire
+		(pts
 			(xy 163.83 76.2) (xy 163.83 80.01)
 		)
@@
 	(wire
 		(pts
+			(xy 120.65 46.99) (xy 120.65 60.96)
+		)
+		(stroke
+			(width 0)
+			(type default)
+		)
+	)
+	(wire
+		(pts
 			(xy 104.14 119.38) (xy 92.71 119.38)
 		)
@@
 	(wire
 		(pts
-			(xy 128.27 49.53) (xy 128.27 60.96)
+			(xy 128.27 46.99) (xy 128.27 60.96)
 		)
 		(stroke
@@
 		)
 	)
+	(wire
+		(pts
+			(xy 90.17 177.8) (xy 104.14 177.8)
+		)
+		(stroke
+			(width 0)
+			(type default)
+		)
+	)
 	(text "Talha Haris and Gavin Wang"
 		(exclude_from_sim no)
@@
 		)
 	)
+	(label "TEG_NEG"
+		(at 102.87 43.18 90)
+		(fields_autoplaced yes)
+		(effects
+			(font
+				(size 1.27 1.27)
+			)
+			(justify left bottom)
+		)
+	)
+	(label "TEG_POS"
+		(at 120.65 46.99 90)
+		(fields_autoplaced yes)
+		(effects
+			(font
+				(size 1.27 1.27)
+			)
+			(justify left bottom)
+		)
+	)
+	(label "TEG_POS"
+		(at 106.68 43.18 90)
+		(fields_autoplaced yes)
+		(effects
+			(font
+				(size 1.27 1.27)
+			)
+			(justify left bottom)
+		)
+	)
+	(label "TEG_NEG"
+		(at 124.46 46.99 90)
+		(fields_autoplaced yes)
+		(effects
+			(font
+				(size 1.27 1.27)
+			)
+			(justify left bottom)
+		)
+	)
 	(symbol
 		(lib_id "power:GND")
@@
 	(symbol
 		(lib_id "power:GNDA")
+		(at 90.17 181.61 0)
+		(unit 1)
+		(exclude_from_sim no)
+		(in_bom yes)
+		(on_board yes)
+		(dnp no)
+		(fields_autoplaced yes)
+		(property "Reference" "#PWR017"
+			(at 90.17 187.96 0)
+			(effects
+				(font
+					(size 1.27 1.27)
+				)
+				(hide yes)
+			)
+		)
+		(property "Value" "GNDA"
+			(at 90.17 186.69 0)
+			(effects
+				(font
+					(size 1.27 1.27)
+				)
+			)
+		)
+		(property "Footprint" ""
+			(at 90.17 181.61 0)
+			(effects
+				(font
+					(size 1.27 1.27)
+				)
+				(hide yes)
+			)
+		)
+		(property "Datasheet" ""
+			(at 90.17 181.61 0)
+			(effects
+				(font
+					(size 1.27 1.27)
+				)
+				(hide yes)
+			)
+		)
+		(property "Description" "Power symbol creates a global label with name \"GNDA\" , analog ground"
+			(at 90.17 181.61 0)
+			(effects
+				(font
+					(size 1.27 1.27)
+				)
+				(hide yes)
+			)
+		)
+		(pin "1"
+		)
+		(instances
+			(project ""
+				(path "/18b83dba-4501-470b-8034-81794e29fc56"
+					(reference "#PWR017")
+					(unit 1)
+				)
+			)
+		)
+	)
+	(symbol
+		(lib_id "power:GNDA")
 		(at 81.28 95.25 270)
 		(unit 1)
@@
 		(lib_name "GM250-127-14-10_1")
 		(lib_id "Energy Harvester:GM250-127-14-10")
-		(at 121.92 43.18 90)
+		(at 105.41 49.53 270)
 		(unit 1)
 		(exclude_from_sim no)
@@
 		(fields_autoplaced yes)
 		(property "Reference" "TEG1"
-			(at 127 42.5449 90)
+			(at 109.22 48.8949 90)
 			(effects
 				(font
@@
 					(italic yes)
 				)
-				(justify right)
+				(justify left)
 			)
 		)
 		(property "Value" "~"
-			(at 127 44.45 90)
+			(at 109.22 50.8 90)
 			(effects
 				(font
@@
 					(italic yes)
 				)
-				(justify right)
+				(justify left)
 			)
 		)
-		(property "Footprint" ""
-			(at 121.92 43.18 0)
+		(property "Footprint" "Connector_Molex:Molex_Micro-Fit_3.0_43650-0200_1x02_P3.00mm_Horizontal"
+			(at 105.41 49.53 0)
 			(effects
 				(font
@@
 		)
 		(property "Datasheet" ""
-			(at 121.92 43.18 0)
+			(at 105.41 49.53 0)
 			(effects
 				(font
@@
 		)
 		(property "Description" ""
-			(at 121.92 43.18 0)
+			(at 105.41 49.53 0)
 			(effects
 				(font
@@
 			)
 		)
-		(pin ""
+		(pin "2"
 		)
-		(pin ""
+		(pin "1"
 		)
 		(instances
@@
 					(unit 1)
 				)
+			)
+		)
+	)
+	(symbol
+		(lib_id "power:GND")
+		(at 104.14 181.61 0)
+		(unit 1)
+		(exclude_from_sim no)
+		(in_bom yes)
+		(on_board yes)
+		(dnp no)
+		(fields_autoplaced yes)
+		(property "Reference" "#PWR018"
+			(at 104.14 187.96 0)
+			(effects
+				(font
+					(size 1.27 1.27)
+				)
+				(hide yes)
+			)
+		)
+		(property "Value" "GND"
+			(at 104.14 186.69 0)
+			(effects
+				(font
+					(size 1.27 1.27)
+				)
+			)
+		)
+		(property "Footprint" ""
+			(at 104.14 181.61 0)
+			(effects
+				(font
+					(size 1.27 1.27)
+				)
+				(hide yes)
+			)
+		)
+		(property "Datasheet" ""
+			(at 104.14 181.61 0)
+			(effects
+				(font
+					(size 1.27 1.27)
+				)
+				(hide yes)
+			)
+		)
+		(property "Description" "Power symbol creates a global label with name \"GND\" , ground"
+			(at 104.14 181.61 0)
+			(effects
+				(font
+					(size 1.27 1.27)
+				)
+				(hide yes)
+			)
+		)
+		(pin "1"
+		)
+		(instances
+			(project ""
+				(path "/18b83dba-4501-470b-8034-81794e29fc56"
+					(reference "#PWR018")
+					(unit 1)
+				)
